File: Wireless_Gyro/Wireless_Gyro.kicad_pcb (KiCad board)
At the start: 2 copper layers, 0 parts

Commit message: Uploading Local changes to fix remote tracking
Parts:
- added BT1: Battery_Cell, Connector_JST:JST_PH_S2B-PH-K_1x02_P2.00mm_Horizontal, F.Cu at (135.0, 140.4)
- added C1: 10uF, Capacitor_SMD:C_0805_2012Metric_Pad1.18x1.45mm_HandSolder, F.Cu at (153.9, 82.2)
- added C2: 100nF, Capacitor_SMD:C_0805_2012Metric_Pad1.18x1.45mm_HandSolder, F.Cu at (156.2, 87.0)
- added C3: 1nF, Capacitor_SMD:C_0805_2012Metric_Pad1.18x1.45mm_HandSolder, F.Cu at (108.8, 95.9)
- added C4: 10uF, Capacitor_SMD:C_0805_2012Metric_Pad1.18x1.45mm_HandSolder, F.Cu at (137.8, 141.5)
- added C5: 10uF, Capacitor_SMD:C_0805_2012Metric_Pad1.18x1.45mm_HandSolder, F.Cu at (170.8, 94.8)
- added C6: 10uF, Capacitor_SMD:C_0805_2012Metric_Pad1.18x1.45mm_HandSolder, F.Cu at (201.0, 116.8)
- added D1: Green, LED_THT:LED_D5.0mm_Clear, F.Cu at (128.6, 104.5)
- added D2: 1N5817, Diode_THT:D_DO-41_SOD81_P10.16mm_Horizontal, F.Cu at (204.2, 115.8)
- added D3: 1N5817, Diode_THT:D_DO-41_SOD81_P10.16mm_Horizontal, F.Cu at (207.6, 115.8)
- added J1: Conn_01x08_Female, Connector_PinHeader_2.54mm:PinHeader_1x08_P2.54mm_Vertical, B.Cu at (220.7, 115.8)
- added J2: Gyro GND, Connector_PinSocket_2.54mm:PinSocket_1x01_P2.54mm_Vertical, F.Cu at (195.2, 105.5)
- added J3: INT-D5, Connector_PinSocket_2.54mm:PinSocket_1x01_P2.54mm_Vertical, F.Cu at (199.8, 105.5)
- added J3: Conn_01x08_Female, Connector_PinHeader_2.54mm:PinHeader_1x08_P2.54mm_Vertical, B.Cu at (197.7, 115.8)
- added J4: 3.3V, Connector_PinSocket_2.54mm:PinSocket_1x01_P2.54mm_Vertical, F.Cu at (174.2, 88.3)
- added J4: Conn_01x06_Female, Connector_PinSocket_2.54mm:PinSocket_1x06_P2.54mm_Vertical, F.Cu at (216.2, 74.2)
- added J5: Conn_01x06_Female, Connector_PinSocket_2.54mm:PinSocket_1x06_P2.54mm_Vertical, F.Cu at (211.6, 74.2)
- added P1: USB_C_Plug_USB2.0, Custom:USB_C_THT, F.Cu at (125.7, 70.3)
- added Q1: IRF7404, Package_SO:SOIC-8_3.9x4.9mm_P1.27mm, F.Cu at (165.5, 87.0)
- added Q2: Q_Dual_NMOS_S1G1D2S2G2D1, Package_TO_SOT_SMD:SOT-23-6_Handsoldering, F.Cu at (149.6, 141.4)
- added R1: 1k, Resistor_SMD:R_0603_1608Metric_Pad0.98x0.95mm_HandSolder, F.Cu at (157.1, 82.1)
- added R10: 470, Resistor_SMD:R_0603_1608Metric_Pad0.98x0.95mm_HandSolder, F.Cu at (153.8, 139.1)
- added R11: 220k, Resistor_SMD:R_0603_1608Metric_Pad0.98x0.95mm_HandSolder, F.Cu at (211.9, 130.6)
- added R2: 1k, Resistor_SMD:R_0603_1608Metric_Pad0.98x0.95mm_HandSolder, F.Cu at (128.7, 110.3)
- added R3: 150m, Resistor_SMD:R_0603_1608Metric_Pad0.98x0.95mm_HandSolder, F.Cu at (160.3, 81.5)
- added R4: 22k, Resistor_SMD:R_0603_1608Metric_Pad0.98x0.95mm_HandSolder, F.Cu at (128.0, 70.3)
- added R5: 22k, Resistor_SMD:R_0603_1608Metric_Pad0.98x0.95mm_HandSolder, F.Cu at (118.3, 90.1)
- added R6: 10k, Resistor_SMD:R_0603_1608Metric_Pad0.98x0.95mm_HandSolder, F.Cu at (116.7, 90.1)
- added R7: 100k, Resistor_SMD:R_0603_1608Metric_Pad0.98x0.95mm_HandSolder, F.Cu at (110.9, 95.9)
- added R8: 10k, Resistor_SMD:R_0603_1608Metric_Pad0.98x0.95mm_HandSolder, F.Cu at (112.6, 95.9)
- added R9: 330, Resistor_SMD:R_0603_1608Metric_Pad0.98x0.95mm_HandSolder, F.Cu at (150.5, 136.2)
- added SW1: SW_SPDT, Connector_PinHeader_2.54mm:PinHeader_1x02_P2.54mm_Vertical, F.Cu at (141.8, 142.5)
- added TH1: 10k, Connector_PinHeader_2.54mm:PinHeader_1x02_P2.54mm_Vertical, F.Cu at (105.6, 94.7)
- added U1: MCP73841, Package_SO:MSOP-10_3x3mm_P0.5mm, F.Cu at (159.4, 87.0)
- added U2: S-8240AAW-I6T1U, Custom:SNT-6A, F.Cu at (154.4, 141.4)
Routing:
- net Net-(BT1-Pad1): track 0.00 -> 32.7 mm
- net +5V: track 0.00 -> 23.1 mm, vias 0 -> 2
- net Net-(C3-Pad1): track 0.00 -> 14.4 mm
- net GND: track 0.00 -> 12.6 mm, vias 0 -> 3
- net Net-(Q1-Pad1): track 0.00 -> 11.0 mm
- net Load: track 0.00 -> 9.88 mm
- net Net-(R9-Pad2): track 0.00 -> 9.03 mm
- net Net-(Q1-Pad4): track 0.00 -> 6.62 mm
- net Net-(C6-Pad2): track 0.00 -> 5.63 mm, vias 0 -> 1
- net Net-(Q2-Pad3): track 0.00 -> 3.75 mm
- net Net-(C2-Pad2): track 0.00 -> 3.71 mm
- net Net-(R1-Pad1): track 0.00 -> 3.24 mm
- net Net-(Q2-Pad2): track 0.00 -> 2.70 mm
- net Net-(Q2-Pad4): track 0.00 -> 2.64 mm
- net Net-(P1-PadA5): track 0.00 -> 2.42 mm
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- added copper zone on In2.Cu, net +5V
- added copper zone on B.Cu, net GND
- added copper zone on F.Cu, net GND
- added copper zone on F.Cu, net Net-(BT1-Pad1)
- added copper zone on In1.Cu, net Net-(C6-Pad2)
- added copper zone on F.Cu, net Net-(Q1-Pad1)
- added copper zone on F.Cu, net Net-(Q2-Pad4)
Other:
- copper layers 2 -> 4
