File: Wireless_Gyro/Wireless_Gyro.kicad_sch (KiCad schematic)
At the start: 21 parts, among them J1 Conn_01x08_Female, J2 Conn_01x08_Female, P1 USB_C_Plug_USB2.0, SW1 SW_SPDT, U1 L6924D013TR

Commit message: Uploading Local changes to fix remote tracking
Parts:
- removed D2: Red, symbol Device:LED
- removed R2: 1k, Resistor_SMD:R_0603_1608Metric_Pad0.98x0.95mm_HandSolder, symbol Device:R
- removed U1: L6924D013TR, Package_DFN_QFN:VQFN-16-1EP_3x3mm_P0.5mm_EP1.68x1.68mm_ThermalVias, symbol Custom_Symbols:L6924D013TR
- added C5: 10uF, Capacitor_SMD:C_0805_2012Metric_Pad1.18x1.45mm_HandSolder, symbol Device:C_Small
- added J2: Gyro GND, Connector_PinSocket_2.54mm:PinSocket_1x01_P2.54mm_Vertical, symbol Connector:Conn_01x01_Female
- added J4, J5: Conn_01x06_Female, Connector_PinSocket_2.54mm:PinSocket_1x06_P2.54mm_Vertical, symbol Connector:Conn_01x06_Female
- added Q1: IRF7404, Package_SO:SOIC-8_3.9x4.9mm_P1.27mm, symbol Transistor_FET:IRF7404
- added Q2: Q_Dual_NMOS_S1G1D2S2G2D1, Package_TO_SOT_SMD:SOT-23-6_Handsoldering, symbol Device:Q_Dual_NMOS_S1G1D2S2G2D1
- added R1: 1k, Resistor_SMD:R_0603_1608Metric_Pad0.98x0.95mm_HandSolder, symbol Device:R
- added R10: 470, Resistor_SMD:R_0603_1608Metric_Pad0.98x0.95mm_HandSolder, symbol Device:R
- added R11: 220k, Resistor_SMD:R_0603_1608Metric_Pad0.98x0.95mm_HandSolder, symbol Device:R
- added R6, R8: 10k, Resistor_SMD:R_0603_1608Metric_Pad0.98x0.95mm_HandSolder, symbol Device:R
- added R7: 100k, Resistor_SMD:R_0603_1608Metric_Pad0.98x0.95mm_HandSolder, symbol Device:R
- added R9: 330, Resistor_SMD:R_0603_1608Metric_Pad0.98x0.95mm_HandSolder, symbol Device:R
- added U1: MCP73841, Package_SO:MSOP-10_3x3mm_P0.5mm, symbol Custom_Symbols:MCP73841
- added U2: S-8240AAW-I6T1U, Custom:SNT-6A, symbol Custom_Symbols:S-8240AAW-I6T1U
- BT1: footprint (none) -> Connector_JST:JST_PH_S2B-PH-K_1x02_P2.00mm_Horizontal
- C1, C3, C4: footprint Capacitor_SMD:C_0603_1608Metric_Pad1.08x0.95mm_HandSolder -> Capacitor_SMD:C_0805_2012Metric_Pad1.18x1.45mm_HandSolder
- C2: value 11.3nF -> 100nF; footprint Capacitor_SMD:C_0603_1608Metric_Pad1.08x0.95mm_HandSolder -> Capacitor_SMD:C_0805_2012Metric_Pad1.18x1.45mm_HandSolder
- C6: renamed from C5; footprint Capacitor_SMD:C_0603_1608Metric_Pad1.08x0.95mm_HandSolder -> Capacitor_SMD:C_0805_2012Metric_Pad1.18x1.45mm_HandSolder
- D1: footprint (none) -> LED_THT:LED_D5.0mm_Clear
- P1: footprint (none) -> Custom:USB_C_THT
- R3: value 15.5k -> 150m
- R4: value 1k -> 22k
- R5: value 50k -> 22k
- TH1: value 50k -> 10k
- renumbered D3 to D2, D4 to D3, J2 to J1, J1 to J3, R1 to R2
Connections:
- net +3.3V: now also C5.1, J4.2 (Pin_2)
- net +5V: now also R2.2, R3.1, R4.1, R1.2, U1.2 (V_{DD}); no longer R2.1
- net GND: now also C2.1, J4.3 (Pin_3), R7.2, R8.2, U1.8 (V_{SS}), U2.4 (VSS); no longer C2.2, C6.2, R3.2, R4.2
- net at R5.1: now also R6.1, U1.5 (TH_{REF}); no longer C3.1
- net at SW1.2 (B): now also Q2.3 (S); no longer J3.2 (Pin_2)
- net at BT1.1 (+), C4.1, D3.2 (A): now also Q1.5 (D), Q1.6 (D), Q1.7 (D), Q1.8 (D), R11.2, R9.1, U1.9 (V_{BAT})
- net at D1.1 (K): now also U1.3 (STAT1)
- net SDA: now reaches J3.5 (Pin_5)
- net SDA: now also J4.5 (Pin_5)
- net SCL: now reaches J3.6 (Pin_6)
- net SCL: now also J4.4 (Pin_4)
- net at D1.2 (A): now also R2.1; no longer R2.2
- net INT: now reaches J1.5 (Pin_5)
- net INT: now also J4.6 (Pin_6)
- net at J1.7 (Pin_7): now also R11.1
- net at P1.A5 (CC): now also R4.2
- net TH: no longer names the net of R5.2, TH1.1
- net TH: now also C3.1, R6.2, R7.1, R8.1, U1.6 (TH_{ERM})
- new net: Q2.6 (G), U2.2 (CO)
- new net: Q2.4 (G), U2.3 (DO)
- new net: R9.2, U2.5 (VDD)
- new net: R10.1, U2.6 (VM)
- new net: C5.2, C6.2, J2.1 (Pin_1), J3.2 (Pin_2), Q2.1 (S), R10.2
- new net: Q1.1 (S), Q1.2 (S), Q1.3 (S), R3.2, U1.1 (SENSE)
- new net: Q1.4 (G), U1.10 (DRV)
- new net: R1.1, U1.4 (EN)
- new net: C2.2, U1.7 (TIMER)
- new net: Q2.2 (D), Q2.5 (D)
- no-connect marks 6 -> 4
Other:
- note added: "ESP and Gyro will be on opposite sides of the PCB"
- note added: "R_{cold} = 27.74k R_{hot} = 3.02k RT_{1} = 6.778k ~ 22k//10k (~1.4% error) RT_{2} = 8.969k ~ 100k//10k (~1.4% error)"
- note added: "Worst Case: ~2W Dissipation"
- note added: "~80mW (1/8W will do) Dissipation"
- moved on the sheet: C1, C3, C6, D1, D2, D3, J1, J3, P1, R2, TH1
